Commit message: hokuyo path fixed

File: leo_description/urdf/sensors/all_sensors.urdf.xacro (robot description, xacro)
@@ -14,5 +14,5 @@
   <!-- Imu -->
   <!-- Hokuyo -->
-  <xacro:include filename="$(find rb1_description)/urdf/sensors/hokuyo.urdf.xacro" />
+  <xacro:include filename="$(find leo_description)/urdf/sensors/hokuyo.urdf.xacro" />
   <!-- Camera -->
 </robot>

File: leo_description/urdf/sensors/hokuyo.urdf.xacro (robot description, xacro)
@@ -28,5 +28,5 @@
         <origin xyz="0 0 -0.05" rpy="0 0 0"/>
         <geometry>
-            <mesh filename="package://rb1_description/meshes/sensors/hokuyo/hokuyo_ust_20lx.dae"/>
+            <mesh filename="package://leo_description/meshes/sensors/hokuyo/hokuyo_ust_20lx.dae"/>
         </geometry>
       </visual>
