Commit message: hokuyo dae

File: leo_description/urdf/sensors/hokuyo.urdf.xacro (robot description, xacro)
@@ -28,5 +28,5 @@
         <origin xyz="0 0 -0.05" rpy="0 0 0"/>
         <geometry>
-            <mesh filename="package://leo_description/meshes/sensors/hokuyo/hokuyo_ust_20lx.dae"/>
+            <mesh filename="package://leo_description/models/hokuyo_ust_20lx.dae"/>
         </geometry>
       </visual>
