Commit message: hokuyo added

File: leo_description/urdf/macros.xacro (robot description, xacro)
@@ -1,4 +1,5 @@
 <?xml version="1.0" encoding="utf-8"?>
 <robot xmlns:xacro="http://www.ros.org/wiki/xacro">
+  <xacro:include filename="$(find leo_description)/urdf/sensors/all_sensors.urdf.xacro" />
   <xacro:macro name="leo"
                params="default_antenna:=true
@@ -385,7 +386,10 @@
         <robot_param>robot_description</robot_param>
         <robot_param_node>robot_state_publisher</robot_param_node>
-        <parameters>package://leo_description/config/controllers.yaml</parameters>
+        <parameters>$(find leo_description)/config/controllers.yaml</parameters>
       </plugin>
     </gazebo>
+    <xacro:sensor_hokuyo prefix="${link_prefix}front_laser" parent="${link_prefix}base_link">
+        <origin xyz="0.105 0.0 0.05" rpy="0 0 0"/>
+    </xacro:sensor_hokuyo>
   </xacro:macro>
   <xacro:macro name="leo_sim"

Commit message: hokuyo moved

File: leo_description/urdf/macros.xacro (robot description, xacro)
@@ -9,4 +9,7 @@
                        joint_prefix:=''
                        imu_translation:='0.0628 -0.0314 -0.0393'">
+    <xacro:sensor_hokuyo prefix="${link_prefix}front_laser" parent="${link_prefix}base_link">
+        <origin xyz="0.105 0.0 0.05" rpy="0 0 0"/>
+    </xacro:sensor_hokuyo>
     <xacro:macro name="rocker_link" params="name">
       <link name="${link_prefix}rocker_${name}_link">
@@ -389,7 +392,4 @@
       </plugin>
     </gazebo>
-    <xacro:sensor_hokuyo prefix="${link_prefix}front_laser" parent="${link_prefix}base_link">
-        <origin xyz="0.105 0.0 0.05" rpy="0 0 0"/>
-    </xacro:sensor_hokuyo>
   </xacro:macro>
   <xacro:macro name="leo_sim"
